File: Projects/DF_ESC/DF_ESC/Design/rev01/rev01_1/Schematics/MOSFET DRIVER.kicad_sch (KiCad schematic)
At the start: 0 parts

Commit message: Update 07
Added the mosfet driver to the schematics
Parts:
- added U2: DRV8302DCA, DCA56_6P35X3P61, symbol 2025-02-11_00-46-13:DRV8302DCA
Other:
- note added: "${TITLE}"
- title: (none) -> MOSFET DRIVER
Changed lines of the file:
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@@
 (kicad_sch (version 20230121) (generator eeschema)
   (paper "A4")
+  (title_block
+    (title "MOSFET DRIVER")
+    (date "2025-02-10")
+  )
+  (text "${TITLE}" (at 111.76 30.48 0)
+    (effects (font (size 5.27 5.27) bold) (justify left bottom))
+  )
+  (symbol (lib_id "2025-02-11_00-46-13:DRV8302DCA") (at 119.38 67.31 0) (unit 1)
+    (in_bom yes) (on_board yes) (dnp no) (fields_autoplaced)
+    (property "Reference" "U2" (at 142.875 57.15 0)
+      (effects (font (size 1.524 1.524)))
+    )
+    (property "Value" "DRV8302DCA" (at 142.875 59.69 0)
+      (effects (font (size 1.524 1.524)))
+    )
+    (property "Footprint" "DCA56_6P35X3P61" (at 116.84 62.23 0)
+      (effects (font (size 1.27 1.27) italic) hide)
+    )
+    (property "Datasheet" "DRV8302DCA" (at 116.84 64.77 0)
+      (effects (font (size 1.27 1.27) italic) hide)
+    )
+    (pin "1")
+    (pin "10")
+    (pin "11")
+    (pin "12")
+    (pin "13")
+    (pin "14")
+    (pin "15")
+    (pin "16")
+    (pin "17")
+    (pin "18")
+    (pin "19")
+    (pin "2")
+    (pin "20")
+    (pin "21")
+    (pin "22")
+    (pin "23")
+    (pin "24")
+    (pin "25")
+    (pin "26")
+    (pin "27")
+    (pin "28")
+    (pin "29")
+    (pin "3")
+    (pin "30")
+    (pin "31")
+    (pin "32")
+    (pin "33")
+    (pin "34")
+    (pin "35")
+    (pin "36")
+    (pin "37")
+    (pin "38")
+    (pin "39")
+    (pin "4")
+    (pin "40")
+    (pin "41")
+    (pin "42")
+    (pin "43")
+    (pin "44")
+    (pin "45")
+    (pin "46")
+    (pin "47")
+    (pin "48")
+    (pin "49")
+    (pin "5")
+    (pin "50")
+    (pin "51")
+    (pin "52")
+    (pin "53")
+    (pin "54")
+    (pin "55")
+    (pin "56")
+    (pin "57")
+    (pin "6")
+    (pin "7")
+    (pin "8")
+    (pin "9")
+    (instances
+      (project "DF_ESC"
+        (path "/e63e39d7-6ac0-4ffd-8aa3-1841a4541b55/7d060fa9-2cfc-44da-bd85-18de38f9a574"
+          (reference "U2") (unit 1)
+        )
+      )
+    )
+  )
 )
